Commit message: fixed test trajectories, changed damping and friction in urdf

File: src/closetbot/urdf/DexArm.urdf.xacro (robot description, xacro)
@@ -945,5 +945,5 @@
     </hardware>
     <joint name="bases">
-      <dynamics damping="10.0" friction="10.0" />
+      <dynamics damping="100.0" friction="100.0" />
       <command_interface name="position">
         <param name="min">-6.28</param>
@@ -954,5 +954,5 @@
     </joint>
     <joint name="B_Rot->In_1">
-      <dynamics damping="10.0" friction="10.0" />
+      <dynamics damping="100.0" friction="100.0" />
       <command_interface name="position">
         <param name="min">-6.28</param>
@@ -963,5 +963,5 @@
     </joint>
     <joint name="In_1->Join">
-      <dynamics damping="10.0" friction="10.0" />
+      <dynamics damping="100.0" friction="100.0" />
       <command_interface name="position">
         <param name="min">-6.28</param>
@@ -972,5 +972,5 @@
     </joint>
     <joint name="Join->In_2">
-      <dynamics damping="10.0" friction="10.0" />
+      <dynamics damping="100.0" friction="100.0" />
       <command_interface name="position">
         <param name="min">-6.28</param>
@@ -981,5 +981,5 @@
     </joint>
     <joint name="In_2->EE">
-      <dynamics damping="10.0" friction="10.0" />
+      <dynamics damping="100.0" friction="100.0" />
       <command_interface name="position">
         <param name="min">-6.28</param>
@@ -990,5 +990,5 @@
     </joint>
     <joint name="Join->Out_1">
-      <dynamics damping="10.0" friction="10.0" />
+      <dynamics damping="100.0" friction="100.0" />
       <command_interface name="position">
         <param name="min">-6.28</param>
@@ -999,5 +999,5 @@
     </joint>
     <joint name="Join->Out_2">
-      <dynamics damping="10.0" friction="10.0" />
+      <dynamics damping="100.0" friction="100.0" />
       <command_interface name="position">
         <param name="min">-6.28</param>
@@ -1008,5 +1008,5 @@
     </joint>
     <!-- <joint name="EE->GripperMount">
-      <dynamics damping="10.0" friction="10.0" />
+      <dynamics damping="100.0" friction="100.0" />
       <command_interface name="position">
         <param name="min">-6.28</param>
@@ -1017,5 +1017,5 @@
     </joint> -->
     <joint name="GripperMount->GripperAxis">
-      <dynamics damping="10.0" friction="10.0" />
+      <dynamics damping="100.0" friction="100.0" />
       <command_interface name="position">
         <param name="min">-6.28</param>
@@ -1026,5 +1026,5 @@
     </joint>
     <joint name="GripperFingerA1->GripperFingerA2">
-      <dynamics damping="10.0" friction="10.0" />
+      <dynamics damping="100.0" friction="100.0" />
       <command_interface name="position">
         <param name="min">-6.28</param>
@@ -1035,5 +1035,5 @@
     </joint>
     <joint name="GripperFingerA2->GripperFingerA3">
-      <dynamics damping="10.0" friction="10.0" />
+      <dynamics damping="100.0" friction="100.0" />
       <command_interface name="position">
         <param name="min">-6.28</param>
@@ -1044,5 +1044,5 @@
     </joint>
     <joint name="GripperFingerA3->GripperFingerA4">
-      <dynamics damping="10.0" friction="10.0" />
+      <dynamics damping="100.0" friction="100.0" />
       <command_interface name="position">
         <param name="min">-6.28</param>
@@ -1053,5 +1053,5 @@
     </joint>
     <joint name="GripperFingerA4->GripperFingerA5">
-      <dynamics damping="10.0" friction="10.0" />
+      <dynamics damping="100.0" friction="100.0" />
       <command_interface name="position">
         <param name="min">-6.28</param>
@@ -1062,5 +1062,5 @@
     </joint>
     <!-- <joint name="GripperAxis->GripperFingerB1">
-      <dynamics damping="10.0" friction="10.0" />
+      <dynamics damping="100.0" friction="100.0" />
       <command_interface name="position">
         <param name="min">-6.28</param>
@@ -1071,5 +1071,5 @@
     </joint>     -->
     <joint name="GripperFingerB1->GripperFingerB2">
-      <dynamics damping="10.0" friction="10.0" />
+      <dynamics damping="100.0" friction="100.0" />
       <command_interface name="position">
         <param name="min">-6.28</param>
@@ -1080,5 +1080,5 @@
     </joint>
     <joint name="GripperFingerB2->GripperFingerB3">
-      <dynamics damping="10.0" friction="10.0" />
+      <dynamics damping="100.0" friction="100.0" />
       <command_interface name="position">
         <param name="min">-6.28</param>
@@ -1089,5 +1089,5 @@
     </joint>
     <joint name="GripperFingerB3->GripperFingerB4">
-      <dynamics damping="10.0" friction="10.0" />
+      <dynamics damping="100.0" friction="100.0" />
       <command_interface name="position">
         <param name="min">-6.28</param>
@@ -1098,5 +1098,5 @@
     </joint>
     <joint name="GripperFingerB4->GripperFingerB5">
-      <dynamics damping="10.0" friction="10.0" />
+      <dynamics damping="100.0" friction="100.0" />
       <command_interface name="position">
         <param name="min">-6.28</param>
@@ -1107,5 +1107,5 @@
     </joint>
     <!-- <joint name="GripperAxis->GripperFingerC1">
-      <dynamics damping="10.0" friction="10.0" />
+      <dynamics damping="100.0" friction="100.0" />
       <command_interface name="position">
         <param name="min">-6.28</param>
@@ -1116,5 +1116,5 @@
     </joint>     -->
     <joint name="GripperFingerC1->GripperFingerC2">
-      <dynamics damping="10.0" friction="10.0" />
+      <dynamics damping="100.0" friction="100.0" />
       <command_interface name="position">
         <param name="min">-6.28</param>
@@ -1125,5 +1125,5 @@
     </joint>
     <joint name="GripperFingerC2->GripperFingerC3">
-      <dynamics damping="10.0" friction="10.0" />
+      <dynamics damping="100.0" friction="100.0" />
       <command_interface name="position">
         <param name="min">-6.28</param>
@@ -1134,5 +1134,5 @@
     </joint>
     <joint name="GripperFingerC3->GripperFingerC4">
-      <dynamics damping="10.0" friction="10.0" />
+      <dynamics damping="100.0" friction="100.0" />
       <command_interface name="position">
         <param name="min">-6.28</param>
@@ -1143,5 +1143,5 @@
     </joint>
     <joint name="GripperFingerC4->GripperFingerC5">
-      <dynamics damping="10.0" friction="10.0" />
+      <dynamics damping="100.0" friction="100.0" />
       <command_interface name="position">
         <param name="min">-6.28</param>
